File: zasilanie.kicad_sch (KiCad schematic)
At the start: 25 parts, among them J1 USB4135-GF-A_REVA, U21 TP4056, U31 FP6291

Commit message: eh
Parts:
- removed R8: 10k, Resistor_SMD:R_0201_0603Metric_Pad0.64x0.40mm_HandSolder, symbol Device:R
- added R: 10k, Resistor_SMD:R_0201_0603Metric_Pad0.64x0.40mm_HandSolder, symbol Device:R
- GREEN2: footprint Library:red diode -> Library:green diode
- renumbered C2 to C, C_Elec8 to C_Elec, L1 to L
Connections:
- net BAT+: now also U31. (EN); no longer U31.4 (EN)
- net GND: now also R.2
- net at J1.B5 (CC2): now also R.1
Changed lines of the file:
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@@
 		(on_board yes)
 		(dnp no)
-		(property "Reference" "C_Elec8"
+		(property "Reference" "C_Elec"
 			(at 79.756 70.104 0)
 			(effects
@@
 			(project "projekt1"
 				(path "/904d1d75-f953-4b81-801a-1eb5237af7a5/d7c7b31c-5e9d-4fbe-918f-cf65aa5b9702"
-					(reference "C_Elec8")
+					(reference "C_Elec")
 					(unit 1)
 				)
@@
 		(dnp no)
 		(fields_autoplaced yes)
-		(property "Reference" "L1"
+		(property "Reference" "L"
 			(at 173.99 107.95 90)
 			(effects
@@
 			(project "projekt1"
 				(path "/904d1d75-f953-4b81-801a-1eb5237af7a5/d7c7b31c-5e9d-4fbe-918f-cf65aa5b9702"
-					(reference "L1")
+					(reference "L")
 					(unit 1)
 				)
@@
 		(pin "2"
 		)
-		(pin "4"
+		(pin ""
 		)
 		(instances
@@
 	(symbol
 		(lib_id "Device:R")
+		(at 36.83 45.72 0)
+		(unit 1)
+		(exclude_from_sim no)
+		(in_bom yes)
+		(on_board yes)
+		(dnp no)
+		(property "Reference" "R"
+			(at 38.608 43.942 0)
+			(effects
+				(font
+					(size 1.27 1.27)
+				)
+				(justify left)
+			)
+		)
+		(property "Value" "10k"
+			(at 38.1 45.72 0)
+			(effects
+				(font
+					(size 1.27 1.27)
+				)
+				(justify left)
+			)
+		)
+		(property "Footprint" "Resistor_SMD:R_0201_0603Metric_Pad0.64x0.40mm_HandSolder"
+			(at 35.052 45.72 90)
+			(effects
+				(font
+					(size 1.27 1.27)
+				)
+				(hide yes)
+			)
+		)
+		(property "Datasheet" "~"
+			(at 36.83 45.72 0)
+			(effects
+				(font
+					(size 1.27 1.27)
+				)
+				(hide yes)
+			)
+		)
+		(property "Description" "Resistor"
+			(at 36.83 45.72 0)
+			(effects
+				(font
+					(size 1.27 1.27)
+				)
+				(hide yes)
+			)
+		)
+		(pin "1"
+		)
+		(pin "2"
+		)
+		(instances
+			(project "projekt1"
+				(path "/904d1d75-f953-4b81-801a-1eb5237af7a5/d7c7b31c-5e9d-4fbe-918f-cf65aa5b9702"
+					(reference "R")
+					(unit 1)
+				)
+			)
+		)
+	)
+	(symbol
+		(lib_id "Device:R")
 		(at 48.26 52.07 0)
 		(unit 1)
@@
 			)
 		)
-		(property "Footprint" "Library:red diode"
+		(property "Footprint" "Library:green diode"
 			(at 100.33 77.47 0)
 			(effects
@@
 		(on_board yes)
 		(dnp no)
-		(property "Reference" "C2"
+		(property "Reference" "C"
 			(at 58.42 49.784 0)
 			(effects
@@
 			(project "projekt1"
 				(path "/904d1d75-f953-4b81-801a-1eb5237af7a5/d7c7b31c-5e9d-4fbe-918f-cf65aa5b9702"
-					(reference "C2")
+					(reference "C")
 					(unit 1)
 				)
@@
 					(unit 1)
 				)
-			)
-		)
-	)
-	(symbol
-		(lib_id "Device:R")
-		(at 36.83 45.72 0)
-		(unit 1)
-		(exclude_from_sim no)
-		(in_bom yes)
-		(on_board yes)
-		(dnp no)
-		(property "Reference" "R8"
-			(at 38.608 43.942 0)
-			(effects
-				(font
-					(size 1.27 1.27)
-				)
-				(justify left)
-			)
-		)
-		(property "Value" "10k"
-			(at 38.1 45.72 0)
-			(effects
-				(font
-					(size 1.27 1.27)
-				)
-				(justify left)
-			)
-		)
-		(property "Footprint" "Resistor_SMD:R_0201_0603Metric_Pad0.64x0.40mm_HandSolder"
-			(at 35.052 45.72 90)
-			(effects
-				(font
-					(size 1.27 1.27)
-				)
-				(hide yes)
-			)
-		)
-		(property "Datasheet" "~"
-			(at 36.83 45.72 0)
-			(effects
-				(font
-					(size 1.27 1.27)
-				)
-				(hide yes)
-			)
-		)
-		(property "Description" "Resistor"
-			(at 36.83 45.72 0)
-			(effects
-				(font
-					(size 1.27 1.27)
-				)
-				(hide yes)
-			)
-		)
-		(pin "1"
-		)
-		(pin "2"
-		)
-		(instances
-			(project "projekt1"
-				(path "/904d1d75-f953-4b81-801a-1eb5237af7a5/d7c7b31c-5e9d-4fbe-918f-cf65aa5b9702"
-					(reference "R8")
-					(unit 1)
-				)
