File: zasilanie modol.kicad_sch (KiCad schematic)
At the start: 25 parts, among them J1 USB4135-GF-A_REVA, U21 TP4056, U31 FP6291

Commit message: latest
Parts:
- added BT1: Battery_Cell, Library:18650, symbol Device:Battery_Cell
- added C3: 100n, Library:C0805F104K1RACAUTO, symbol Device:C
- added NMOS1, NMOS2: Q_NMOS, Library:RTF016N05MOSFET, symbol Device:Q_NMOS
- added R12: 6m, Library:WFCP04026L000FE66, symbol Device:R
- added R13: 20, Resistor_SMD:R_0201_0603Metric_Pad0.64x0.40mm_HandSolder, symbol Device:R
- added R14: 300, Resistor_SMD:R_0201_0603Metric_Pad0.64x0.40mm_HandSolder, symbol Device:R
- added R15: 1k, Resistor_SMD:R_0201_0603Metric_Pad0.64x0.40mm_HandSolder, symbol Device:R
- added U2: BQ298010, Library:BQ29801, symbol M5Stamp:BQ298010
- C_Elec1, C_Elec2, C_Elec3, C_Elec4, C_Elec5, C_Elec6, C_Elec7: footprint Capacitor_SMD:C_Elec_4x5.4 -> Library:C_ELEC10u5PH2D5
- R1, R8: value 10k -> 5k1
- renumbered J1 to USB1
Connections:
- net BAT+: now also BT1.1 (+), NMOS1.S, R13.1, R14.1; no longer C_Elec1.1, C_Elec2.1, C_Elec3.1, C_Elec4.1, L1.1, U31.4 (EN), U31.5 (VCC)
- net GND: now also R12.2, U2.4 (CS), U2.5 (CTR)
- net VBUS: now also C1.1, USB1.B9 (VBUS_B)
- net VCC renamed 5V
- new net: R13.2, U2.1 (BAT)
- new net: C3.1, R14.2, U2.2 (VDD)
- new net: R15.2, U2.6 (PACK)
- new net: NMOS2.G, U2.7 (DSG)
- new net: NMOS1.G, U2.8 (CHG)
- new net: NMOS1.D, NMOS2.D
- new net: C_Elec1.1, C_Elec2.1, C_Elec3.1, C_Elec4.1, L1.1, NMOS2.S, R15.1, U31.4 (EN), U31.5 (VCC)
- new net BAT-: BT1.2 (-), C3.2, R12.1, U2.3 (VSS)
Other:
- moved on the sheet: C2, C_Elec1, C_Elec2, C_Elec3, C_Elec4, C_Elec5, C_Elec6, C_Elec7, C_Elec8, GREEN2, L1, R1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
