File: projekt1.kicad_pcb (KiCad board)
At the start: 2 copper layers, 44 parts, among them J1 USB4135-GF-A_REVA, U1 M5STAMP-S3, U2 RV-3028-C7, U21 TP4056, U3 SCD42, U31 FP6291

Commit message: eh
Parts:
- removed C0805F104K1RACAUTOC1, C0805F104K1RACAUTOC2, C0805F104K1RACAUTOC3, C0805F104K1RACAUTOC4, C0805F104K1RACAUTOC5, C0805F104K1RACAUTOC6, C0805F104K1RACAUTOC7, C0805F104K1RACAUTOC8: 100n, Library:C0805F104K1RACAUTO
- removed LCXHF3030QKT4R7MNRL1: 4.7uH, Library:LCXHF3030QKT4R7MNR
- removed REF** (x2): 18650 holder, Library:18650
- removed SCCR12E105SRBC1, SCCR12E105SRBC2: 1F, Library:SCCR12E105SRB
- removed SMD0201R1, SMD0201R2, SMD0201R3, SMD0201R4, SMD0201R5, SMD0201R6: 10k, Resistor_SMD:R_0201_0603Metric_Pad0.64x0.40mm_HandSolder
- removed SMD0201R10, SMD0201R11: 600, Resistor_SMD:R_0201_0603Metric_Pad0.64x0.40mm_HandSolder
- removed SMD0201R12: 1.2k, Resistor_SMD:R_0201_0603Metric_Pad0.64x0.40mm_HandSolder
- removed SMD0201R13: 48k, Resistor_SMD:R_0201_0603Metric_Pad0.64x0.40mm_HandSolder
- removed SMD0201R14: 88k, Resistor_SMD:R_0201_0603Metric_Pad0.64x0.40mm_HandSolder
- removed SMD0201R7: 12k, Resistor_SMD:R_0201_0603Metric_Pad0.64x0.40mm_HandSolder
- removed SMD0201R8, SMD0201R9: 5k1, Resistor_SMD:R_0201_0603Metric_Pad0.64x0.40mm_HandSolder
- removed SMD:C_Elec_4x5.4C1, SMD:C_Elec_4x5.4C2, SMD:C_Elec_4x5.4C3, SMD:C_Elec_4x5.4C4, SMD:C_Elec_4x5.4C5, SMD:C_Elec_4x5.4C6, SMD:C_Elec_4x5.4C7, SMD:C_Elec_4x5.4C8: 10uF, Capacitor_SMD:C_Elec_4x5.4
- removed U1: M5STAMP-S3, Library:M5STAMP S3
- removed U2: RV-3028-C7, Package_SON:MicroCrystal_C7_SON-8_1.5x3.2mm_P0.9mm
- removed U3: SCD42, Library:SCD42_SEN
- added C1: 100n, Library:C0805F104K1RACAUTO, F.Cu at (71.0, 101.5)
- added C2: 100n, Library:C0805F104K1RACAUTO, F.Cu at (71.0, 105.5)
- added C_Elec1: 10uF, Capacitor_SMD:C_Elec_4x5.4, F.Cu at (95.5, 90.5)
- added C_Elec2: 10uF, Capacitor_SMD:C_Elec_4x5.4, F.Cu at (95.5, 96.3)
- added C_Elec3: 10uF, Capacitor_SMD:C_Elec_4x5.4, F.Cu at (95.5, 102.2)
- added C_Elec4: 10uF, Capacitor_SMD:C_Elec_4x5.4, F.Cu at (95.5, 108.0)
- added C_Elec5: 10uF, Capacitor_SMD:C_Elec_4x5.4, F.Cu at (65.0, 93.0)
- added C_Elec6: 10uF, Capacitor_SMD:C_Elec_4x5.4, F.Cu at (65.0, 79.0)
- added C_Elec7: 10uF, Capacitor_SMD:C_Elec_4x5.4, F.Cu at (65.0, 86.0)
- added C_Elec8: 10uF, Capacitor_SMD:C_Elec_4x5.4, F.Cu at (74.0, 110.5)
- added L1: 4.7uH, Library:LCXHF3030QKT4R7MNR, F.Cu at (87.0, 99.0)
- added R1: 10k, Resistor_SMD:R_0201_0603Metric_Pad0.64x0.40mm_HandSolder, F.Cu at (72.0, 102.5)
- added R2: 600, Resistor_SMD:R_0201_0603Metric_Pad0.64x0.40mm_HandSolder, F.Cu at (83.5, 104.2)
- added R3: 600, Resistor_SMD:R_0201_0603Metric_Pad0.64x0.40mm_HandSolder, F.Cu at (83.5, 106.0)
- added R4: 1k2, Resistor_SMD:R_0201_0603Metric_Pad0.64x0.40mm_HandSolder, F.Cu at (74.5, 98.0)
- added R5: 48k, Resistor_SMD:R_0201_0603Metric_Pad0.64x0.40mm_HandSolder, F.Cu at (87.5, 90.0)
- added R6: 88k, Resistor_SMD:R_0201_0603Metric_Pad0.64x0.40mm_HandSolder, F.Cu at (83.5, 93.0)
- added R7: 12k, Resistor_SMD:R_0201_0603Metric_Pad0.64x0.40mm_HandSolder, F.Cu at (83.5, 94.5)
- added R8: 10k, Resistor_SMD:R_0201_0603Metric_Pad0.64x0.40mm_HandSolder, F.Cu at (71.5, 104.0)
- GREEN2: footprint Library:SSL-LX2573SGD -> Library:red diode
- RED2: footprint Library:SSL-LX2573SRD -> Library:red diode
- moved J1 64.0 mm to (63.5, 103.5), turned to -90 degrees
- moved U21 41.5 mm to (79.5, 98.5)
- moved D2 41.0 mm to (73.4, 89.5)
- moved RED2 40.9 mm to (79.5, 106.5)
- moved GREEN2 40.7 mm to (79.5, 103.5)
- moved U31 34.5 mm to (87.0, 93.5), turned to -90 degrees
Connections:
- U31 pad 4: (no net) -> BAT+
Routing:
- net SCL: track 49.3 -> 0.00 mm, vias 2 -> 0
- net BAT-: track 145.4 -> 114.0 mm
- net Net-(U31-FB): track 29.2 -> 1.96 mm, vias 2 -> 0
- net BAT+: track 70.1 -> 44.8 mm, vias 0 -> 2
- net Net-(U2-VBACKUP): track 15.3 -> 0.00 mm, vias 1 -> 0
- net VCC: track 54.4 -> 40.8 mm, vias 2 -> 0
- net Net-(U31-OC): track 12.3 -> 2.65 mm, vias 2 -> 0
- net VBUS: track 42.2 -> 34.1 mm, vias 5 -> 2
- net Net-(U21-PROG): track 9.85 -> 3.41 mm, vias 2 -> 0
- net Net-(D2-A): track 26.7 -> 21.3 mm, vias 5 -> 2
- net Net-(U21-CHRG#): track 15.4 -> 10.0 mm, vias 2 -> 0
- net Net-(J1-CC1): track 0.00 -> 5.27 mm
- net Net-(J1-CC2): track 0.00 -> 4.56 mm
- net Net-(U21-STDBY#): track 11.0 -> 6.49 mm, vias 2 -> 0
- net Net-(J1-VBUS_B): track 0.00 -> 3.52 mm
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Other:
- board outline added: 41.5 x 39 mm

Commit message: latest
Parts:
- removed C1, C2: 100n, Library:C0805F104K1RACAUTO
- removed C_Elec1, C_Elec2, C_Elec3, C_Elec4, C_Elec5, C_Elec6, C_Elec7: 10uF, Capacitor_SMD:C_Elec_4x5.4
- removed D2: D1, Diode_THT:D_DO-41_SOD81_P10.16mm_Horizontal
- removed J1: USB4135-GF-A_REVA, Connector_USB:USB_C_Receptacle_GCT_USB4135-GF-A_6P_TopMnt_Horizontal
- removed L1: 4.7uH, Library:LCXHF3030QKT4R7MNR
- removed R1, R8: 10k, Resistor_SMD:R_0201_0603Metric_Pad0.64x0.40mm_HandSolder
- removed R2, R3: 600, Resistor_SMD:R_0201_0603Metric_Pad0.64x0.40mm_HandSolder
- removed R4: 1k2, Resistor_SMD:R_0201_0603Metric_Pad0.64x0.40mm_HandSolder
- removed R5: 48k, Resistor_SMD:R_0201_0603Metric_Pad0.64x0.40mm_HandSolder
- removed R6: 88k, Resistor_SMD:R_0201_0603Metric_Pad0.64x0.40mm_HandSolder
- removed R7: 12k, Resistor_SMD:R_0201_0603Metric_Pad0.64x0.40mm_HandSolder
- added BT1: Battery_Cell, Library:18650, F.Cu at (119.0, 93.0)
- added C100n: 100n, Library:C0805F104K1RACAUTO, F.Cu at (107.2, 81.5)
- added C100n: 100n, Library:C0805F104K1RACAUTO, F.Cu at (100.1, 72.5)
- added C100n: 100n, Library:C0805F104K1RACAUTO, F.Cu at (147.2, 70.0)
- added C100n: 100n, Library:C0805F104K1RACAUTO, F.Cu at (75.0, 62.0)
- added C100n: 100n, Library:C0805F104K1RACAUTO, F.Cu at (149.0, 56.5)
- added C100n: 100n, Library:C0805F104K1RACAUTO, F.Cu at (112.4, 81.5)
- added C100n: 100n, Library:C0805F104K1RACAUTO, F.Cu at (113.0, 62.0)
- added C100n: 100n, Library:C0805F104K1RACAUTO, F.Cu at (84.5, 70.0)
- added C100n: 100n, Library:C0805F104K1RACAUTO, F.Cu at (86.0, 67.2)
- added C100n: 100n, Library:C0805F104K1RACAUTO, F.Cu at (157.5, 56.5)
- added C10uF: 10uF, Library:C_ELEC10u5PH2D5, F.Cu at (127.0, 56.8)
- added C10uF: 10uF, Library:C_ELEC10u5PH2D5, F.Cu at (137.5, 57.0)
- added C10uF: 10uF, Library:C_ELEC10u5PH2D5, F.Cu at (121.2, 76.5)
- added C10uF: 10uF, Library:C_ELEC10u5PH2D5, F.Cu at (121.2, 66.0)
- added C10uF: 10uF, Library:C_ELEC10u5PH2D5, F.Cu at (116.5, 56.2)
- added C10uF: 10uF, Library:C_ELEC10u5PH2D5, F.Cu at (131.8, 66.8)
- added C10uF: 10uF, Library:C_ELEC10u5PH2D5, F.Cu at (131.5, 77.0)
- added C1F: 1F, Library:SCCR12E105SRB, F.Cu at (108.3, 78.2)
- added C1F: 1F, Library:SCCR12E105SRB, F.Cu at (108.3, 75.2)
- added FeRAM: ~, Package_SO:SOP-8_3.9x4.9mm_P1.27mm, F.Cu at (78.5, 71.0)
- added L4.7uH: 4.7uH, Library:LCXHF3030QKT4R7MNR, F.Cu at (138.8, 73.5)
- added NMOS1: Q_NMOS, Library:RTF016N05MOSFET, F.Cu at (144.5, 67.5)
- added NMOS2: Q_NMOS, Library:RTF016N05MOSFET, F.Cu at (141.5, 69.2)
- added R10k: 10k, Resistor_SMD:R_0201_0603Metric_Pad0.64x0.40mm_HandSolder, F.Cu at (101.0, 74.5)
- added R15: 1k, Resistor_SMD:R_0201_0603Metric_Pad0.64x0.40mm_HandSolder, F.Cu at (151.0, 70.8)
- added R1k2: 1k2, Resistor_SMD:R_0201_0603Metric_Pad0.64x0.40mm_HandSolder, F.Cu at (157.5, 60.0)
- added R20: 20, Resistor_SMD:R_0201_0603Metric_Pad0.64x0.40mm_HandSolder, F.Cu at (149.8, 65.2)
- added R22k: 12k, Resistor_SMD:R_0201_0603Metric_Pad0.64x0.40mm_HandSolder, F.Cu at (150.0, 70.4)
- added R300: 300, Resistor_SMD:R_0201_0603Metric_Pad0.64x0.40mm_HandSolder, F.Cu at (147.5, 67.8)
- added R48k: 48k, Resistor_SMD:R_0201_0603Metric_Pad0.64x0.40mm_HandSolder, F.Cu at (143.2, 72.5)
- added R4K7: 4k7, Resistor_SMD:R_0201_0603Metric_Pad0.64x0.40mm_HandSolder, F.Cu at (99.2, 78.2)
- added R4k7: 4k7, Resistor_SMD:R_0201_0603Metric_Pad0.64x0.40mm_HandSolder, F.Cu at (88.0, 55.5)
- added R4k7: 4k7, Resistor_SMD:R_0201_0603Metric_Pad0.64x0.40mm_HandSolder, F.Cu at (99.2, 75.8)
- added R4k7: 4k7, Resistor_SMD:R_0201_0603Metric_Pad0.64x0.40mm_HandSolder, F.Cu at (113.0, 49.5)
- added R4k7: 4k7, Resistor_SMD:R_0201_0603Metric_Pad0.64x0.40mm_HandSolder, F.Cu at (112.4, 51.5)
- added R5k1: 5k1, Resistor_SMD:R_0201_0603Metric_Pad0.64x0.40mm_HandSolder, F.Cu at (155.0, 57.0)
- added R5k1: 5k1, Resistor_SMD:R_0201_0603Metric_Pad0.64x0.40mm_HandSolder, F.Cu at (153.1, 57.5)
- added R600: 600, Resistor_SMD:R_0201_0603Metric_Pad0.64x0.40mm_HandSolder, F.Cu at (154.0, 67.2)
- added R600: 600, Resistor_SMD:R_0201_0603Metric_Pad0.64x0.40mm_HandSolder, F.Cu at (152.8, 67.2)
- added R6m: 6m, Library:WFCP04026L000FE66, F.Cu at (151.8, 72.8)
- added R88k: 88k, Resistor_SMD:R_0201_0603Metric_Pad0.64x0.40mm_HandSolder, F.Cu at (150.0, 72.9)
- added SCD41: SCD42, Library:SCD42_SEN, F.Cu at (81.0, 58.7)
- added U1: M5STAMP-S3, Library:M5STAMP S3, F.Cu at (100.0, 59.8)
- added U2: BQ298010, Library:BQ29801, F.Cu at (149.4, 68.2)
- added U4: RV-3028-C7, Package_SON:MicroCrystal_C7_SON-8_1.5x3.2mm_P0.9mm, F.Cu at (101.4, 77.5)
- added USB1: USB4135-GF-A_REVA, Connector_USB:USB_C_Receptacle_GCT_USB4135-GF-A_6P_TopMnt_Horizontal, F.Cu at (154.5, 51.5)
- added schottky: D1, Diode_THT:D_DO-41_SOD81_P10.16mm_Horizontal, F.Cu at (149.2, 77.2)
- moved C_Elec8 87.9 mm to (146.0, 60.0), turned to 90 degrees
- moved RED2 87.2 mm to (157.5, 67.5), turned to 180 degrees
- moved GREEN2 84.5 mm to (157.5, 71.0), turned to 180 degrees
- moved U21 82.2 mm to (153.4, 62.5), turned to -90 degrees
- moved U31 62.7 mm to (146.2, 73.0), turned to 0 degrees
Connections:
- net BAT- renamed GND
- U21 pad 5: BAT+ -> /Untitled Sheet/BAT+
- U31 pad 4: BAT+ -> Net-(U31-EN)
- U31 pad 5: BAT+ -> Net-(U31-EN)
Routing:
- net GND: track 114.0 -> 277.7 mm, vias 0 -> 4
- net /Untitled Sheet/BAT+: track 0.00 -> 89.8 mm, vias 0 -> 2
- net 5V: track 0.00 -> 86.3 mm, vias 0 -> 2
- net SCL: track 0.00 -> 84.2 mm, vias 0 -> 4
- net SDA: track 0.00 -> 82.7 mm, vias 0 -> 4
- net VCC: track 40.8 -> 110.8 mm, vias 0 -> 4
- net Net-(U31-EN): track 0.00 -> 59.1 mm, vias 0 -> 2
- net /SPICSO: track 0.00 -> 51.2 mm, vias 0 -> 4
- net /SPIWP: track 0.00 -> 48.4 mm, vias 0 -> 4
- net /SPIHD: track 0.00 -> 46.2 mm, vias 0 -> 4
- net BAT+: track 44.8 -> 0.00 mm, vias 2 -> 0
- net /SPID: track 0.00 -> 43.1 mm, vias 0 -> 6
- net /SPICLK: track 0.00 -> 39.2 mm, vias 0 -> 4
- net /SPIQ: track 0.00 -> 36.8 mm, vias 0 -> 4
- net /RTC_INT#: track 0.00 -> 34.2 mm, vias 0 -> 2
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Other:
- board outline removed

Commit message: aaaaaaaaaaaaaaaaaaaaaaaaaaaaaaa
Parts:
- removed C100n (x10): 100n, Library:C0805F104K1RACAUTO
- removed C10uF (x7): 10uF, Library:C_ELEC10u5PH2D5
- removed C1F (x2): 1F, Library:SCCR12E105SRB
- removed C_Elec8: 10uF, Capacitor_SMD:C_Elec_4x5.4
- removed FeRAM: ~, Package_SO:SOP-8_3.9x4.9mm_P1.27mm
- removed GREEN2, RED2: LED, Library:red diode
- removed L4.7uH: 4.7uH, Library:LCXHF3030QKT4R7MNR
- removed R10k: 10k, Resistor_SMD:R_0201_0603Metric_Pad0.64x0.40mm_HandSolder
- removed R1k2: 1k2, Resistor_SMD:R_0201_0603Metric_Pad0.64x0.40mm_HandSolder
- removed R20: 20, Resistor_SMD:R_0201_0603Metric_Pad0.64x0.40mm_HandSolder
- removed R22k: 12k, Resistor_SMD:R_0201_0603Metric_Pad0.64x0.40mm_HandSolder
- removed R300: 300, Resistor_SMD:R_0201_0603Metric_Pad0.64x0.40mm_HandSolder
- removed R48k: 48k, Resistor_SMD:R_0201_0603Metric_Pad0.64x0.40mm_HandSolder
- removed R4K7, R4k7 (x4): 4k7, Resistor_SMD:R_0201_0603Metric_Pad0.64x0.40mm_HandSolder
- removed R5k1 (x2): 5k1, Resistor_SMD:R_0201_0603Metric_Pad0.64x0.40mm_HandSolder
- removed R600 (x2): 600, Resistor_SMD:R_0201_0603Metric_Pad0.64x0.40mm_HandSolder
- removed R6m: 6m, Library:WFCP04026L000FE66
- removed R88k: 88k, Resistor_SMD:R_0201_0603Metric_Pad0.64x0.40mm_HandSolder
- removed SCD41: SCD42, Library:SCD42_SEN
- removed U21: TP4056, Package_SO:HSOP-8-1EP_3.9x4.9mm_P1.27mm_EP2.3x2.3mm_ThermalVias
- removed U31: FP6291, Library:SOT23-6L
- removed schottky: D1, Diode_THT:D_DO-41_SOD81_P10.16mm_Horizontal
- added C1: 100n, Library:C0805F104K1RACAUTO, F.Cu at (173.8, 37.7)
- added C10: 100n, Library:C0805F104K1RACAUTO, F.Cu at (132.9, 61.8)
- added C11: 100n, Library:C0805F104K1RACAUTO, F.Cu at (132.9, 63.9)
- added C12: 100n, Library:C0805F104K1RACAUTO, F.Cu at (132.9, 66.0)
- added C13: 100n, Library:C0805F104K1RACAUTO, F.Cu at (132.9, 68.1)
- added C14: 10uF, Capacitor_SMD:C_Elec_4x5.4, F.Cu at (128.7, 88.7)
- added C15: 100n, Library:C0805F104K1RACAUTO, F.Cu at (132.9, 70.2)
- added C2: 100n, Library:C0805F104K1RACAUTO, F.Cu at (173.8, 39.8)
- added C3: 100n, Library:C0805F104K1RACAUTO, F.Cu at (173.8, 41.9)
- added C4: 100n, Library:C0805F104K1RACAUTO, F.Cu at (173.8, 44.0)
- added C5: 1F, Library:SCCR12E105SRB, F.Cu at (160.7, 62.8)
- added C6: 1F, Library:SCCR12E105SRB, F.Cu at (160.7, 65.9)
- added C7: 100n, Library:C0805F104K1RACAUTO, F.Cu at (173.8, 46.1)
- added C8: 100n, Library:C0805F104K1RACAUTO, F.Cu at (173.8, 48.2)
- added C9: 100n, Library:C0805F104K1RACAUTO, F.Cu at (173.8, 50.3)
- added CE1: 10uF, Capacitor_SMD:CP_Elec_6.3x5.4, F.Cu at (130.3, 35.0)
- added CE2: 10uF, Capacitor_SMD:CP_Elec_6.3x5.4, F.Cu at (130.3, 43.1)
- added D1: D1, Diode_THT:D_DO-41_SOD81_P10.16mm_Horizontal, F.Cu at (126.8, 58.6)
- added GREEN1: LED, Library:red diode, F.Cu at (129.3, 80.1)
- added JP1: SolderJumper_2_Bridged, Jumper:SolderJumper-2_P1.3mm_Bridged_Pad1.0x1.5mm, F.Cu at (173.6, 64.9)
- added L1: 4.7uH, Library:LCXHF3030QKT4R7MNR, F.Cu at (132.2, 98.0)
- added R1: 4k7, Resistor_SMD:R_0201_0603Metric_Pad0.64x0.40mm_HandSolder, F.Cu at (177.6, 37.5)
- added R10: 20, Resistor_SMD:R_0201_0603Metric_Pad0.64x0.40mm_HandSolder, F.Cu at (126.4, 66.8)
- added R11: 6m, Library:WFCP04026L000FE66, F.Cu at (126.6, 102.1)
- added R12: 1k, Resistor_SMD:R_0201_0603Metric_Pad0.64x0.40mm_HandSolder, F.Cu at (126.4, 68.6)
- added R13: 600, Resistor_SMD:R_0201_0603Metric_Pad0.64x0.40mm_HandSolder, F.Cu at (126.4, 70.3)
- added R14: 600, Resistor_SMD:R_0201_0603Metric_Pad0.64x0.40mm_HandSolder, F.Cu at (129.2, 61.6)
- added R16: 12k, Resistor_SMD:R_0201_0603Metric_Pad0.64x0.40mm_HandSolder, F.Cu at (129.2, 65.1)
- added R17: 48k, Resistor_SMD:R_0201_0603Metric_Pad0.64x0.40mm_HandSolder, F.Cu at (129.2, 66.8)
- added R18: 1k2, Resistor_SMD:R_0201_0603Metric_Pad0.64x0.40mm_HandSolder, F.Cu at (129.2, 68.6)
- added R2: 4k7, Resistor_SMD:R_0201_0603Metric_Pad0.64x0.40mm_HandSolder, F.Cu at (177.6, 39.3)
- added R3: 4k7, Resistor_SMD:R_0201_0603Metric_Pad0.64x0.40mm_HandSolder, F.Cu at (177.6, 41.0)
- added R4: 10k, Resistor_SMD:R_0201_0603Metric_Pad0.64x0.40mm_HandSolder, F.Cu at (177.6, 42.8)
- added R5: 4k7, Resistor_SMD:R_0201_0603Metric_Pad0.64x0.40mm_HandSolder, F.Cu at (177.6, 44.5)
- added R6: 4k7, Resistor_SMD:R_0201_0603Metric_Pad0.64x0.40mm_HandSolder, F.Cu at (177.6, 46.3)
- added R7: 5k1, Resistor_SMD:R_0201_0603Metric_Pad0.64x0.40mm_HandSolder, F.Cu at (126.4, 61.6)
- added R8: 5k1, Resistor_SMD:R_0201_0603Metric_Pad0.64x0.40mm_HandSolder, F.Cu at (126.4, 63.3)
- added R9: 300, Resistor_SMD:R_0201_0603Metric_Pad0.64x0.40mm_HandSolder, F.Cu at (126.4, 65.1)
- added RED1: LED, Library:red diode, F.Cu at (129.3, 84.1)
- added U3: RV-3028-C7, Package_SON:MicroCrystal_C7_SON-8_1.5x3.2mm_P0.9mm, F.Cu at (166.9, 64.0)
- added U5: BQ298010, Library:BQ29801, F.Cu at (136.3, 97.5)
- added U6: FP6291, Library:SOT23-6L, F.Cu at (127.3, 98.5)
- added U7: TP4056, Package_SO:HSOP-8-1EP_3.9x4.9mm_P1.27mm_EP2.3x2.3mm_ThermalVias, F.Cu at (129.2, 74.6)
- R15: value 1k -> 88k
- U2: value BQ298010 -> 249-MB85RS256BPFGNE1; footprint Library:BQ29801 -> Package_SO:SOP-8_3.9x4.9mm_P1.27mm
- U4: value RV-3028-C7 -> SCD42; footprint Package_SON:MicroCrystal_C7_SON-8_1.5x3.2mm_P0.9mm -> Library:SCD42_SEN
- moved U4 78.6 mm to (177.3, 57.2)
- moved U1 60.8 mm to (159.8, 49.0), turned to 0 degrees
- moved NMOS1 31.7 mm to (126.7, 93.8), turned to 0 degrees
- moved NMOS2 27.0 mm to (130.2, 93.8)
- moved R15 23.0 mm to (129.2, 63.3), turned to 0 degrees
- moved USB1 22.5 mm to (132.0, 51.9), turned to 0 degrees
- moved BT1 20.1 mm to (114.4, 73.4), turned to 0 degrees
- moved U2 4.74 mm to (152.4, 64.7)
Connections:
- NMOS1 pad G: Net-(U2-CHG) -> Net-(U5-CHG)
- NMOS2 pad G: Net-(U2-DSG) -> Net-(U5-DSG)
- NMOS2 pad S: Net-(U31-EN) -> GND
- R15 pad 1: Net-(U31-EN) -> 5V
- R15 pad 2: Net-(U2-PACK) -> Net-(U6-FB)
- U1 pad 1: /SPIHD -> unconnected-(U1-G1-Pad1)
- U1 pad 2: /SPICSO -> unconnected-(U1-G2-Pad2)
- U1 pad 4: /SPID -> /SPICSO
- U1 pad 5: unconnected-(U1-G5-Pad5) -> /SPIHD
- U1 pad 6: /SPICLK -> /SPID
- U1 pad 7: /SPIQ -> /SPICLK
- U1 pad 9: unconnected-(U1-G9-Pad9) -> /SPIQ
- U2 pad 1: Net-(U2-BAT) -> /SPICSO
- U2 pad 2: Net-(U2-VDD) -> /SPID
- U2 pad 3: /Untitled Sheet/BAT- -> /SPIWP
- U2 pad 5: GND -> /SPIQ
- U2 pad 6: Net-(U2-PACK) -> /SPICLK
- U2 pad 7: Net-(U2-DSG) -> /SPIHD
- U2 pad 8: Net-(U2-CHG) -> VCC
- U4 pad 6: Net-(U4-VBACKUP) -> GND
Routing:
- net GND: track 277.7 -> 0.00 mm, vias 4 -> 0
- net VCC: track 110.8 -> 0.00 mm, vias 4 -> 0
- net /Untitled Sheet/BAT+: track 89.8 -> 0.00 mm, vias 2 -> 0
- net 5V: track 86.3 -> 0.00 mm, vias 2 -> 0
- net SCL: track 84.2 -> 0.00 mm, vias 4 -> 0
- net SDA: track 82.7 -> 0.00 mm, vias 4 -> 0
- net Net-(U31-EN): track 59.1 -> 0.00 mm, vias 2 -> 0
- net /SPICSO: track 51.2 -> 0.00 mm, vias 4 -> 0
- net /SPIWP: track 48.4 -> 0.00 mm, vias 4 -> 0
- net /SPIHD: track 46.2 -> 0.00 mm, vias 4 -> 0
- net /SPID: track 43.1 -> 0.00 mm, vias 6 -> 0
- net /SPICLK: track 39.2 -> 0.00 mm, vias 4 -> 0
- net VBUS: track 38.0 -> 0.00 mm, vias 2 -> 0
- net /SPIQ: track 36.8 -> 0.00 mm, vias 4 -> 0
- net /RTC_INT#: track 34.2 -> 0.00 mm, vias 2 -> 0
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