File: projekt1.kicad_sch (KiCad schematic)
At the start: 17 parts, among them U1 M5STAMP-S3, U2 RV-3028-C7, U3 SCD42

Commit message: eh
Parts:
- removed SMD0201R4, SMD0201R5, SMD0201R6: 10k, Resistor_SMD:R_0201_0603Metric_Pad0.64x0.40mm_HandSolder, symbol Device:R
- added R10, R11, R9: 10k, Resistor_SMD:R_0201_0603Metric_Pad0.64x0.40mm_HandSolder, symbol Device:R
Connections:
- net SCL: now also R10.2
- net SDA: now also R9.2
- net VCC: now also R10.1, R11.1, R9.1
- net at U1.22 (EN): now also R11.2

Commit message: update
Parts:
- removed C0805F104K1RACAUTOC5, C0805F104K1RACAUTOC6: 100n, Library:C0805F104K1RACAUTO, symbol Device:C
- removed U3: SCD42, Library:SCD42_SEN, symbol M5Stamp:SCD42
Other:
- sheet Untitled Sheet renamed zasilanie
- added sheet czujnik (czujnik.sch.kicad_sch)

Commit message: latest
Parts:
- added C0805F104K1RACAUTOC3, C0805F104K1RACAUTOC5, C0805F104K1RACAUTOC6: 100n, Library:C0805F104K1RACAUTO, symbol Device:C
- added FeRAM1: ~, Package_SO:SOP-8_3.9x4.9mm_P1.27mm, symbol M5Stamp:249-MB85RS256BPFGNE1
- added U3: SCD42, Library:SCD42_SEN, symbol M5Stamp:SCD42
- R10, R11, R9, SMD0201R2, SMD0201R3: value 10k -> 4k7
- renumbered U2 to U4
Connections:
- net GND: now also C0805F104K1RACAUTOC3.2, C0805F104K1RACAUTOC5.2, C0805F104K1RACAUTOC6.2, FeRAM1.4 (GND), U3.20 (GND), U3.6 (GND)
- net RTC_INT#: now also U1.23 (G11); no longer U1.5 (G5)
- net SCL: now also U3.9 (SCL)
- net SDA: now also U3.10 (SDA)
- net VCC: now also U1.28 (3V3), C0805F104K1RACAUTOC3.1, C0805F104K1RACAUTOC5.1, C0805F104K1RACAUTOC6.1, FeRAM1.8 (VDD), U3.19 (VDDH), U3.7 (VDD); no longer C0805F104K1RACAUTOC7.1, U1.13 (5V)
- net SPIHD: now reaches U1.1 (G1)
- net SPIHD: now also FeRAM1.7 (HOLD#)
- net SPICSO: now reaches U1.2 (G2)
- net SPICSO: now also FeRAM1.1 (CS#)
- net SPID: now reaches U1.4 (G4)
- net SPID: now also FeRAM1.2 (SO)
- net SPICLK: now reaches U1.6 (G6)
- net SPICLK: now also FeRAM1.6 (SCK)
- net SPIQ: now reaches U1.7 (G7)
- net SPIQ: now also FeRAM1.5 (SI)
- net SPIWP: now reaches U1.8 (G8)
- net SPIWP: now also FeRAM1.3 (WP#)
- new net 5V: C0805F104K1RACAUTOC7.1, U1.13 (5V)
Other:
- sheet zasilanie renamed Untitled Sheet
- removed sheet czujnik
- moved on the sheet: C0805F104K1RACAUTOC1, C0805F104K1RACAUTOC2, C0805F104K1RACAUTOC8, R11, SCCR12E105SRBC1, SCCR12E105SRBC2, SMD0201R1, SMD0201R2, SMD0201R3, U4

Commit message: aaaaaaaaaaaaaaaaaaaaaaaaaaaaaaa
Parts:
- added JP1: SolderJumper_2_Bridged, Jumper:SolderJumper-2_P1.3mm_Bridged_Pad1.0x1.5mm, symbol Jumper:SolderJumper_2_Bridged
- U2: renamed from FeRAM1; value ~ -> 249-MB85RS256BPFGNE1
- renumbered C0805F104K1RACAUTOC7 to C1, C0805F104K1RACAUTOC3 to C2, C0805F104K1RACAUTOC8 to C3, C0805F104K1RACAUTOC1 to C4, SCCR12E105SRBC1 to C5, SCCR12E105SRBC2 to C6, C0805F104K1RACAUTOC2 to C7, C0805F104K1RACAUTOC6 to C8, C0805F104K1RACAUTOC5 to C9, R10 to R1, R9 to R2, R11 to R3, SMD0201R1 to R4, SMD0201R2 to R5, SMD0201R3 to R6, U4 to U3, U3 to U4
Connections:
- net SPICLK: now also U1.7 (G7); no longer U1.6 (G6)
- net SPICSO: now also U1.4 (G4); no longer U1.2 (G2)
- net SPID: now also U1.6 (G6); no longer U1.4 (G4)
- net SPIHD: now also U1.5 (G5); no longer U1.1 (G1)
- net SPIQ: now also U1.9 (G9); no longer U1.7 (G7)
- net VCC: now also JP1.2 (B); no longer R1.1, R2.1
- new net: JP1.1 (A), R1.1, R2.1
Other:
- moved on the sheet: C1, C2, C3, C4, C5, C6, C7, C8, C9, R1, R2, R3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
